Commit message: Refactor: Restructure repository and update documentation

File: software/common/altair_description/urdf/altair.urdf (robot description, URDF)
Before this commit: robot altair_hexacopter, 2 links, 1 joints
Links:
- added link arm_1; visual box size=0.25 0.02 0.02
- added link arm_2; visual box size=0.25 0.02 0.02
- added link arm_3; visual box size=0.25 0.02 0.02
- added link arm_4; visual box size=0.25 0.02 0.02
- added link arm_5; visual box size=0.25 0.02 0.02
- added link arm_6; visual box size=0.25 0.02 0.02
- added link rotor_2; visual cylinder length=0.01 radius=0.1
- added link rotor_3; visual cylinder length=0.01 radius=0.1
- added link rotor_4; visual cylinder length=0.01 radius=0.1
- added link rotor_5; visual cylinder length=0.01 radius=0.1
- added link rotor_6; visual cylinder length=0.01 radius=0.1
- added link tilt_1_link; visual cylinder length=0.04 radius=0.02
- added link tilt_2_link; visual cylinder length=0.04 radius=0.02
- added link tilt_3_link; visual cylinder length=0.04 radius=0.02
- added link tilt_4_link; visual cylinder length=0.04 radius=0.02
- added link tilt_5_link; visual cylinder length=0.04 radius=0.02
- added link tilt_6_link; visual cylinder length=0.04 radius=0.02
- link base_link: geometry collision cylinder length=0.05 radius=0.15; visual cylinder length=0.05 radius=0.15
Joints:
- added joint arm_1_joint: type fixed, parent base_link, child arm_1, origin xyz=0 0 0 rpy=0 0 0
- added joint arm_2_joint: type fixed, parent base_link, child arm_2, origin xyz=0 0 0 rpy=0 0 1.0472
- added joint arm_3_joint: type fixed, parent base_link, child arm_3, origin xyz=0 0 0 rpy=0 0 2.0944
- added joint arm_4_joint: type fixed, parent base_link, child arm_4, origin xyz=0 0 0 rpy=0 0 3.14159
- added joint arm_5_joint: type fixed, parent base_link, child arm_5, origin xyz=0 0 0 rpy=0 0 4.1888
- added joint arm_6_joint: type fixed, parent base_link, child arm_6, origin xyz=0 0 0 rpy=0 0 5.2360
- added joint rotor_2_joint: type continuous, parent tilt_2_link, child rotor_2, origin xyz=0 0 0.03 rpy=0 0 0, axis 0 0 1
- added joint rotor_3_joint: type continuous, parent tilt_3_link, child rotor_3, origin xyz=0 0 0.03 rpy=0 0 0, axis 0 0 1
- added joint rotor_4_joint: type continuous, parent tilt_4_link, child rotor_4, origin xyz=0 0 0.03 rpy=0 0 0, axis 0 0 1
- added joint rotor_5_joint: type continuous, parent tilt_5_link, child rotor_5, origin xyz=0 0 0.03 rpy=0 0 0, axis 0 0 1
- added joint rotor_6_joint: type continuous, parent tilt_6_link, child rotor_6, origin xyz=0 0 0.03 rpy=0 0 0, axis 0 0 1
- added joint tilt_1_joint: type revolute, parent arm_1, child tilt_1_link, origin xyz=0.25 0 0 rpy=0 0 0, axis 1 0 0, limit lower=-1.57 upper=1.57 effort=5.0 velocity=5.0
- added joint tilt_2_joint: type revolute, parent arm_2, child tilt_2_link, origin xyz=0.25 0 0 rpy=0 0 0, axis 1 0 0, limit lower=-1.57 upper=1.57 effort=5.0 velocity=5.0
- added joint tilt_3_joint: type revolute, parent arm_3, child tilt_3_link, origin xyz=0.25 0 0 rpy=0 0 0, axis 1 0 0, limit lower=-1.57 upper=1.57 effort=5.0 velocity=5.0
- added joint tilt_4_joint: type revolute, parent arm_4, child tilt_4_link, origin xyz=0.25 0 0 rpy=0 0 0, axis 1 0 0, limit lower=-1.57 upper=1.57 effort=5.0 velocity=5.0
- added joint tilt_5_joint: type revolute, parent arm_5, child tilt_5_link, origin xyz=0.25 0 0 rpy=0 0 0, axis 1 0 0, limit lower=-1.57 upper=1.57 effort=5.0 velocity=5.0
- added joint tilt_6_joint: type revolute, parent arm_6, child tilt_6_link, origin xyz=0.25 0 0 rpy=0 0 0, axis 1 0 0, limit lower=-1.57 upper=1.57 effort=5.0 velocity=5.0
- joint rotor_1_joint: axis (none) -> 0 0 1; origin xyz=0.25 0 0 rpy=0 0 0 -> xyz=0 0 0.03 rpy=0 0 0; parent base_link -> tilt_1_link; type fixed -> continuous
